Commit message: feat(control): control/feedback works for 2 servos

File: champi_description/urdf/arm_description.urdf.xacro (robot description, xacro)
@@ -17,8 +17,24 @@
     </visual>
   </link>
-  <!-- Joint -->
+  <!-- Link 3 -->
+  <link name="link3">
+    <visual>
+      <geometry>
+        <cylinder length="1" radius="0.05"/>
+      </geometry>
+    </visual>
+  </link>
+  <!-- Joint1 -->
   <joint name="joint1" type="revolute">
     <parent link="link1"/>
     <child link="link2"/>
+    <origin xyz="0 0 1" rpy="0 0 0"/>
+    <axis xyz="0 1 0"/>
+    <limit lower="-1.57" upper="1.57" effort="100.0" velocity="0.5"/>
+  </joint>
+  <!-- Joint2 -->
+  <joint name="joint2" type="revolute">
+    <parent link="link2"/>
+    <child link="link3"/>
     <origin xyz="0 0 1" rpy="0 0 0"/>
     <axis xyz="0 1 0"/>
@@ -35,7 +51,11 @@
         <param name="id">13</param>
         <command_interface name="position"/>
-        <command_interface name="velocity"/>
         <state_interface name="position"/>
-        <state_interface name="velocity"/>
+        <state_interface name="effort"/>
+      </joint>
+      <joint name="joint2">
+        <param name="id">11</param>
+        <command_interface name="position"/>
+        <state_interface name="position"/>
         <state_interface name="effort"/>
       </joint>
