Commit message: lidar CPU ok

File: champi_description/urdf/champi.urdf (robot description, URDF)
Before this commit: robot my_robot, 3 links, 2 joints
Links:
- removed link ldlidar_base
- added link base_laser, mass 1
Joints:
- joint base_to_lidar: child ldlidar_base -> base_laser; origin xyz=0 0 0.3 rpy=0 0 0 -> xyz=0 0 0.3 rpy=0 0 1.57

Commit message: push before homologation

File: champi_description/urdf/champi.urdf (robot description, URDF)
Before this commit: robot my_robot, 3 links, 2 joints
Joints:
- joint base_to_camera: origin xyz=0.082, 0.015, 0.315 rpy=0.000, 0.805, 0.010 -> xyz=0.082 0.015 0.315 rpy=0.000 0.805 0.010

Commit message: new extrinsic calibration

File: champi_description/urdf/champi.urdf (robot description, URDF)
Before this commit: robot my_robot, 3 links, 2 joints
Joints:
- joint base_to_camera: origin xyz=0.082 0.015 0.315 rpy=0.000 0.805 0.010 -> xyz=0.082 0.012 0.320 rpy=0.006 0.802 -0.030
